File: schematics/PSLab.sch (KiCad schematic (older format))
At the start: 183 parts, among them J1 DoublePins, J11 Li-Ion Battery, J2 Power Pins, J3 Wave Generator, J4 I2C, J5 I2C, J6 ESP01, J7 UART, J8 Battery Switch, J9 SPI, P1 SDCard, Q1 MMBT3906, Q2 MMBT3904, Q3 MMBT3906, SW1 BOOT, SW2 MCLR Reset, SW3 USB_C - Generic, U1 FP6291, U10 TL082, U11 TL082, U12 MCP4728, U13 MCP6S21, U14 MCP6S21, U15 CP2102N, U16 SP0503BAHT, U17 IP5189T, U2 74HC126, U3 PIC24EP256GP204, U4 DS1307Z+, U5 TP7660H, U6 HT7333-A, U7 LM324, U8 TL082, U9 TL082, X2 32.768 kHz, Y1 12 MHz

Commit message: Temp2
Parts:
- L2: footprint Inductor_SMD:L_0603_1608Metric -> Inductor_SMD:L_Taiyo-Yuden_MD-2020
Connections:
- no-connect marks 36 -> 35
Changed lines of the file:
@@
 Data
 89 50 4E 47 0D 0A 1A 0A 00 00 00 0D 49 48 44 52 00 00 02 08 00 00 00 CC 08 03 00 00 00 21 C4 AB
-DA 00 00 00 03 73 42 49 54 08 08 08 DB E1 4F E0 00 00 03 00 50 4C 54 45 02 00 00 FF FF E2 79 5D
+DA 00 00 00 03 73 42 49 54 08 08 08 DB E1 4F E0 00 00 03 00 50 4C 54 45 01 00 00 FF FF E2 79 5D
 9D 28 5D A5 28 7D CE E2 FF FF 81 5D B6 A5 EA FF C6 99 A5 28 99 E2 FF EA D6 59 5D C2 C6 FF FF 59
 B6 F2 FF FF F2 A5 7D A5 28 5D C6 E2 B6 B6 81 CE FF FF CE C6 81 7D D6 55 5D A1 59 7D BE F6 F6 F6
@@
 F6 99 D2 CE 40 9D D6 EA EE F6 40 5D A5 28 5D BA 7D D2 DE 55 AE DE 28 75 C2 CA DA EA 99 AA B6 65
 C2 DE 85 A5 CA 4C 4C 4C A1 A1 A1 3C 3C 3C 61 65 69 A5 B2 BE 85 A1 CE 91 99 A1 EE F2 F2 7D 81 81
-B6 BE C6 91 91 91 7D 7D 81 50 79 B6 C2 C2 C2 99 B2 7D 5D B6 DE FA FA FA 4A AB 90 C2 00 00 00 01
+B6 BE C6 91 91 91 7D 7D 81 50 79 B6 C2 C2 C2 99 B2 7D 5D B6 DE FA FA FA 76 CF DF 8C 00 00 00 01
 74 52 4E 53 00 40 E6 D8 66 00 00 15 08 49 44 41 54 78 9C ED 9D 7B 80 15 D5 79 C0 67 99 A5 31 A6
 26 05 83 EC 2E FB 76 60 9B 44 F6 01 BB CA 43 77 F7 C6 18 1F 10 31 36 1B 5D 4C 82 69 D6 24 D6 A0
@@
 Text Notes 15050 650  0    39   ~ 8
 Sine Wave Generator
-Wire Notes Line
-	5325 13775 5350 13775
 $Comp
 L Device:R R27
@@
 Wire Wire Line
 	6475 4200 6800 4200
-NoConn ~ 4100 15300
 $Comp
 L Device:CP1_Small C12
@@
 F 0 "L2" V 3685 4300 50  0000 C CNN
 F 1 "4.7uH" V 3594 4300 50  0000 C CNN
-F 2 "Inductor_SMD:L_0603_1608Metric" H 3500 4300 50  0001 C CNN
-F 3 "~" H 3500 4300 50  0001 C CNN
+F 2 "Inductor_SMD:L_Taiyo-Yuden_MD-2020" H 3500 4300 50  0001 C CNN
+F 3 "https://item.szlcsc.com/992539.html SMNR201610-4R7MT" H 3500 4300 50  0001 C CNN
 	1    3500 4300
 	0    -1   -1   0

Commit message: Temp3
Parts:
- SW3: footprint Connector_USB:USB_C_Receptacle_XKB_U262-16XN-4BVC11 -> incremental_library:USB_C_Receptacle_12pin_SMT
Changed lines of the file:
@@
 F 0 "SW3" V 2050 2250 39  0000 L CNN
 F 1 "USB_C - Generic" V 2050 -125 39  0000 L CNN
-F 2 "Connector_USB:USB_C_Receptacle_XKB_U262-16XN-4BVC11" H 2650 1275 50  0001 C CNN
+F 2 "incremental_library:USB_C_Receptacle_12pin_SMT" H 2650 1275 50  0001 C CNN
 F 3 "https://cdn.sparkfun.com/assets/8/6/b/4/5/A40-00119-A52-12.pdf" H 2650 1275 50  0001 C CNN
 F 4 "USB - Type C Female 16 SMT" H 2500 1275 50  0001 C CNN "Description"
@@
 Data
 89 50 4E 47 0D 0A 1A 0A 00 00 00 0D 49 48 44 52 00 00 02 08 00 00 00 CC 08 03 00 00 00 21 C4 AB
-DA 00 00 00 03 73 42 49 54 08 08 08 DB E1 4F E0 00 00 03 00 50 4C 54 45 01 00 00 FF FF E2 79 5D
+DA 00 00 00 03 73 42 49 54 08 08 08 DB E1 4F E0 00 00 03 00 50 4C 54 45 02 00 00 FF FF E2 79 5D
 9D 28 5D A5 28 7D CE E2 FF FF 81 5D B6 A5 EA FF C6 99 A5 28 99 E2 FF EA D6 59 5D C2 C6 FF FF 59
 B6 F2 FF FF F2 A5 7D A5 28 5D C6 E2 B6 B6 81 CE FF FF CE C6 81 7D D6 55 5D A1 59 7D BE F6 F6 F6
@@
 F6 99 D2 CE 40 9D D6 EA EE F6 40 5D A5 28 5D BA 7D D2 DE 55 AE DE 28 75 C2 CA DA EA 99 AA B6 65
 C2 DE 85 A5 CA 4C 4C 4C A1 A1 A1 3C 3C 3C 61 65 69 A5 B2 BE 85 A1 CE 91 99 A1 EE F2 F2 7D 81 81
-B6 BE C6 91 91 91 7D 7D 81 50 79 B6 C2 C2 C2 99 B2 7D 5D B6 DE FA FA FA 76 CF DF 8C 00 00 00 01
+B6 BE C6 91 91 91 7D 7D 81 50 79 B6 C2 C2 C2 99 B2 7D 5D B6 DE FA FA FA 4A AB 90 C2 00 00 00 01
 74 52 4E 53 00 40 E6 D8 66 00 00 15 08 49 44 41 54 78 9C ED 9D 7B 80 15 D5 79 C0 67 99 A5 31 A6
 26 05 83 EC 2E FB 76 60 9B 44 F6 01 BB CA 43 77 F7 C6 18 1F 10 31 36 1B 5D 4C 82 69 D6 24 D6 A0
@@
 F 1 "IP5189T" H 2800 4064 37  0000 C CNN
 F 2 "Package_DFN_QFN:QFN-24-1EP_4x4mm_P0.5mm_EP2.6x2.6mm" H 2900 2300 37  0001 C CNN
-F 3 "" H 4500 2600 37  0001 C CNN
+F 3 "http://www.injoinic.com/wwwroot/uploads/files/20200220/3642884e4c0184d6c0173a5193cd56ce.pdf" H 4500 2600 37  0001 C CNN
 	1    2600 4000
 	1    0    0    -1

Commit message: Temp4
Parts:
- removed C43: 0.1uF, Capacitor_SMD:C_0603_1608Metric, symbol Device:C
- removed C44: 10uF, Capacitor_SMD:C_0603_1608Metric, symbol Device:C
- removed U15: CP2102N, Package_DFN_QFN:QFN-24-1EP_4x4mm_P0.5mm_EP2.6x2.6mm, symbol PSLab:CP2102
- added C43: 0.1uF, Capacitor_SMD:C_0603_1608Metric, symbol Device:C_Small
- added C44: 10uF, Capacitor_SMD:C_0603_1608Metric, symbol Device:C_Small
- added U15: CP2102N-xxx-xQFN20x, PSLab:QFN-20_EP_3x3_Pitch0.5mm, symbol PSLab:CP2102N-xxx-xQFN20x
- L1: footprint Inductor_SMD:L_0603_1608Metric -> Inductor_SMD:L_Taiyo-Yuden_MD-2020
- L3: value 3.3uH -> 4.7uH; footprint Inductor_SMD:L_0603_1608Metric -> Inductor_SMD:L_Taiyo-Yuden_MD-2020
Connections:
- net +3V3: no longer R51.2
- net +5V: now also U15.7 (VregIn)
- net D+: now also U15.4 (D+)
- net D-: now also U15.5 (D-)
- net GND: now also C43.2, C44.2, U15.12 (GND), U15.21 (GND), U15.3 (GND)
- net VBusSense: now also U15.8 (VBUS)
- net MRxD: no longer names the net of R54.1
- net MRxD: now also U15.17 (RXD)
- net MTxD: no longer names the net of R55.1
- net MTxD: now also U15.18 (TXD)
- net UARTReset: no longer names the net of R51.1
- net UARTReset: now also U15.9 (RSTb)
- new net CP2102_Vreg: C43.1, C44.1, R51.2, U15.6 (VDD)
- no-connect marks 35 -> 31
Other:
- moved on the sheet: R48, R51, R54, R55, R58
