File: schematics/PSLab.sch (KiCad schematic (older format))
At the start: 183 parts, among them J1 DoublePins, J11 Li-Ion Battery, J2 Power Pins, J3 Wave Generator, J4 I2C, J5 I2C, J6 ESP01, J7 UART, J8 Battery Switch, J9 SPI, P1 SDCard, Q1 MMBT3906, Q2 MMBT3904, Q3 MMBT3906, SW1 BOOT, SW2 MCLR Reset, SW3 USB_C - Generic, U1 FP6291, U10 TL082, U11 TL082, U12 MCP4728, U13 MCP6S21, U14 MCP6S21, U15 CP2102N-xxx-xQFN20x, U16 SP0503BAHT, U17 IP5189T, U2 74HC126, U3 PIC24EP256GP204, U4 DS1307Z+, U5 TP7660H, U6 HT7333-A, U7 LM324, U8 TL082, U9 TL082, X2 32.768 kHz, Y1 12 MHz

Commit message: Temp5
Parts:
- removed D6: LL4148, Diode_SMD:D_MiniMELF, symbol Device:D
Connections:
- wire segments 500 -> 501
Other:
- moved on the sheet: D5
Changed lines of the file:
@@
 	1    0    0    -1
 $EndComp
-Text GLabel 8125 9125 1    40   Input ~ 0
+Text GLabel 8200 9400 2    40   Input ~ 0
 +5V
-Text GLabel 7825 9125 1    40   Output ~ 0
+Text GLabel 7900 9000 2    40   Output ~ 0
 RGB
 $Comp
-L Device:D D6
-U 1 1 5F978449
-P 8125 9275
-F 0 "D6" V 8171 9195 39  0000 R CNN
-F 1 "LL4148" V 8080 9195 39  0000 R CNN
-F 2 "Diode_SMD:D_MiniMELF" H 8125 9275 50  0001 C CNN
-F 3 "https://www.mouser.fi/datasheet/2/395/LL4148_SERIES_J15-1918261.pdf" H 8125 9275 50  0001 C CNN
-F 4 "General Purpose diode" H 8125 9275 50  0001 C CNN "Description"
-F 5 "LL4448 L0" H 8125 9275 50  0001 C CNN "Mfr No."
-F 6 "0.11" H 8125 9275 50  0001 C CNN "Price"
-F 7 "LL4448 L0" H 8125 9275 50  0001 C CNN "PartNumber"
-	1    8125 9275
-	0    -1   -1   0
-$EndComp
-$Comp
 L power:PWR_FLAG #FLG0106
 U 1 1 5FA4B8DD
-P 8125 9425
-F 0 "#FLG0106" H 8125 9500 50  0001 C CNN
-F 1 "PWR_FLAG" H 8125 9598 39  0001 C CNN
-F 2 "" H 8125 9425 50  0001 C CNN
-F 3 "~" H 8125 9425 50  0001 C CNN
-	1    8125 9425
+P 8100 9400
+F 0 "#FLG0106" H 8100 9475 50  0001 C CNN
+F 1 "PWR_FLAG" H 8100 9573 39  0001 C CNN
+F 2 "" H 8100 9400 50  0001 C CNN
+F 3 "~" H 8100 9400 50  0001 C CNN
+	1    8100 9400
 	-1   0    0    1
 $EndComp
@@
 L LED:WS2812B D5
 U 1 1 5F65D829
-P 7825 9425
-F 0 "D5" V 7575 9225 39  0000 L CNN
-F 1 "WS2812B" V 8075 9475 39  0000 L CNN
-F 2 "LED_SMD:LED_WS2812B_PLCC4_5.0x5.0mm_P3.2mm" H 7875 9125 50  0001 L TNN
-F 3 "https://www.mouser.fi/datasheet/2/737/4684_WS2812B_2020_V1_3_EN-1900866.pdf" H 7925 9050 50  0001 L TNN
-F 4 "RGB LED with integrated controller" H 7825 9425 50  0001 C CNN "Description"
-F 5 "WS2812B" H 7825 9425 50  0001 C CNN "Mfr No."
-F 6 "3.35" H 7825 9425 50  0001 C CNN "Price"
-F 7 "WS2812B" H 7825 9425 50  0001 C CNN "PartNumber"
-	1    7825 9425
+P 7800 9400
+F 0 "D5" V 7550 9200 39  0000 L CNN
+F 1 "WS2812B" V 8050 9450 39  0000 L CNN
+F 2 "LED_SMD:LED_WS2812B_PLCC4_5.0x5.0mm_P3.2mm" H 7850 9100 50  0001 L TNN
+F 3 "https://www.mouser.fi/datasheet/2/737/4684_WS2812B_2020_V1_3_EN-1900866.pdf" H 7900 9025 50  0001 L TNN
+F 4 "RGB LED with integrated controller" H 7800 9400 50  0001 C CNN "Description"
+F 5 "WS2812B" H 7800 9400 50  0001 C CNN "Mfr No."
+F 6 "3.35" H 7800 9400 50  0001 C CNN "Price"
+F 7 "WS2812B" H 7800 9400 50  0001 C CNN "PartNumber"
+	1    7800 9400
 	0    1    1    0
 $EndComp
@@
 Data
 89 50 4E 47 0D 0A 1A 0A 00 00 00 0D 49 48 44 52 00 00 02 08 00 00 00 CC 08 03 00 00 00 21 C4 AB
-DA 00 00 00 03 73 42 49 54 08 08 08 DB E1 4F E0 00 00 03 00 50 4C 54 45 02 00 00 FF FF E2 79 5D
+DA 00 00 00 03 73 42 49 54 08 08 08 DB E1 4F E0 00 00 03 00 50 4C 54 45 01 00 00 FF FF E2 79 5D
 9D 28 5D A5 28 7D CE E2 FF FF 81 5D B6 A5 EA FF C6 99 A5 28 99 E2 FF EA D6 59 5D C2 C6 FF FF 59
 B6 F2 FF FF F2 A5 7D A5 28 5D C6 E2 B6 B6 81 CE FF FF CE C6 81 7D D6 55 5D A1 59 7D BE F6 F6 F6
@@
 F6 99 D2 CE 40 9D D6 EA EE F6 40 5D A5 28 5D BA 7D D2 DE 55 AE DE 28 75 C2 CA DA EA 99 AA B6 65
 C2 DE 85 A5 CA 4C 4C 4C A1 A1 A1 3C 3C 3C 61 65 69 A5 B2 BE 85 A1 CE 91 99 A1 EE F2 F2 7D 81 81
-B6 BE C6 91 91 91 7D 7D 81 50 79 B6 C2 C2 C2 99 B2 7D 5D B6 DE FA FA FA 4A AB 90 C2 00 00 00 01
+B6 BE C6 91 91 91 7D 7D 81 50 79 B6 C2 C2 C2 99 B2 7D 5D B6 DE FA FA FA 76 CF DF 8C 00 00 00 01
 74 52 4E 53 00 40 E6 D8 66 00 00 15 08 49 44 41 54 78 9C ED 9D 7B 80 15 D5 79 C0 67 99 A5 31 A6
 26 05 83 EC 2E FB 76 60 9B 44 F6 01 BB CA 43 77 F7 C6 18 1F 10 31 36 1B 5D 4C 82 69 D6 24 D6 A0
@@
 Wire Notes Line
 	7150 11075 8675 11075
-Connection ~ 8125 9425
-NoConn ~ 7825 9725
+NoConn ~ 7800 9700
 $Comp
 L power:GND #PWR?
@@
 L power:GND #PWR?
 U 1 1 6331EC1D
-P 7500 9450
+P 7500 9400
 AR Path="/5ED254D7/6331EC1D" Ref="#PWR?"  Part="1"
 AR Path="/6331EC1D" Ref="#PWR036"  Part="1"
-F 0 "#PWR036" H 7500 9200 50  0001 C CNN
-F 1 "GND" H 7500 9300 39  0000 C CNN
-F 2 "" H 7500 9450 50  0001 C CNN
-F 3 "" H 7500 9450 50  0001 C CNN
-	1    7500 9450
+F 0 "#PWR036" H 7500 9150 50  0001 C CNN
+F 1 "GND" H 7500 9250 39  0000 C CNN
+F 2 "" H 7500 9400 50  0001 C CNN
+F 3 "" H 7500 9400 50  0001 C CNN
+	1    7500 9400
 	1    0    0    -1
 $EndComp
-Wire Wire Line
-	7500 9450 7500 9425
-Wire Wire Line
-	7500 9425 7525 9425
 Wire Notes Line
 	5325 6725 8675 6725
@@
 Wire Wire Line
 	7600 1600 7700 1600
+Connection ~ 8100 9400
+Wire Wire Line
+	7800 9000 7800 9100
+Wire Wire Line
+	7800 9000 7900 9000
+Wire Wire Line
+	8100 9400 8200 9400
 $EndSCHEMATC

Commit message: Temp6
Parts:
- removed C10, C8: 33pF, Capacitor_SMD:C_0603_1608Metric, symbol Device:C
- added C10, C8: 12pF, Capacitor_SMD:C_0603_1608Metric, symbol Device:C_Small
Connections:
- wire segments 501 -> 496
Other:
- moved on the sheet: C13, C17, C21, C4, R1, R10, R12, R2, R3, R49, R56, R57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

Commit message: chore: replace switch to SPST_3x4x2.5
Parts:
- removed SW1: BOOT, Button_Switch_SMD:SW_SPST_B3U-1000P, symbol Switch:SW_Push
- removed SW2: MCLR Reset, Button_Switch_SMD:SW_SPST_B3U-1000P, symbol Switch:SW_Push
- added SW1, SW2: SW_MEC_5E, PSLab:button_SPST_3x4x2.5, symbol Switch:SW_MEC_5E
Connections:
- wire segments 496 -> 494
Other:
- moved on the sheet: C10, C3, C5, C8

Commit message: Temp7
Parts:
- added R63: 51k, Resistor_SMD:R_0603_1608Metric, symbol Device:R_Small
- added SW3: SW_MEC_5E, PSLab:button_SPST_3x4x2.5, symbol Switch:SW_MEC_5E
Connections:
- wire segments 494 -> 509
Other:
- moved on the sheet: R61
Changed lines of the file:
@@
 Data
 89 50 4E 47 0D 0A 1A 0A 00 00 00 0D 49 48 44 52 00 00 02 08 00 00 00 CC 08 03 00 00 00 21 C4 AB
-DA 00 00 00 03 73 42 49 54 08 08 08 DB E1 4F E0 00 00 03 00 50 4C 54 45 01 00 00 FF FF E2 79 5D
+DA 00 00 00 03 73 42 49 54 08 08 08 DB E1 4F E0 00 00 03 00 50 4C 54 45 02 00 00 FF FF E2 79 5D
 9D 28 5D A5 28 7D CE E2 FF FF 81 5D B6 A5 EA FF C6 99 A5 28 99 E2 FF EA D6 59 5D C2 C6 FF FF 59
 B6 F2 FF FF F2 A5 7D A5 28 5D C6 E2 B6 B6 81 CE FF FF CE C6 81 7D D6 55 5D A1 59 7D BE F6 F6 F6
@@
 F6 99 D2 CE 40 9D D6 EA EE F6 40 5D A5 28 5D BA 7D D2 DE 55 AE DE 28 75 C2 CA DA EA 99 AA B6 65
 C2 DE 85 A5 CA 4C 4C 4C A1 A1 A1 3C 3C 3C 61 65 69 A5 B2 BE 85 A1 CE 91 99 A1 EE F2 F2 7D 81 81
-B6 BE C6 91 91 91 7D 7D 81 50 79 B6 C2 C2 C2 99 B2 7D 5D B6 DE FA FA FA 76 CF DF 8C 00 00 00 01
+B6 BE C6 91 91 91 7D 7D 81 50 79 B6 C2 C2 C2 99 B2 7D 5D B6 DE FA FA FA 4A AB 90 C2 00 00 00 01
 74 52 4E 53 00 40 E6 D8 66 00 00 15 08 49 44 41 54 78 9C ED 9D 7B 80 15 D5 79 C0 67 99 A5 31 A6
 26 05 83 EC 2E FB 76 60 9B 44 F6 01 BB CA 43 77 F7 C6 18 1F 10 31 36 1B 5D 4C 82 69 D6 24 D6 A0
@@
 L Device:R_Small R61
 U 1 1 61CE626C
-P 2000 4900
-F 0 "R61" H 2059 4946 50  0000 L CNN
-F 1 "200k" H 2059 4855 50  0000 L CNN
-F 2 "Resistor_SMD:R_0603_1608Metric" H 2000 4900 50  0001 C CNN
-F 3 "~" H 2000 4900 50  0001 C CNN
-	1    2000 4900
+P 1400 4800
+F 0 "R61" H 1459 4846 50  0000 L CNN
+F 1 "200k" H 1459 4755 50  0000 L CNN
+F 2 "Resistor_SMD:R_0603_1608Metric" H 1400 4800 50  0001 C CNN
+F 3 "~" H 1400 4800 50  0001 C CNN
+	1    1400 4800
 	1    0    0    -1
 $EndComp
-Wire Wire Line
-	2000 4800 2300 4800
 $Comp
 L power:GND #PWR0105
@@
 L power:GND #PWR0150
 U 1 1 61D98315
-P 2000 5000
-F 0 "#PWR0150" H 2000 4750 50  0001 C CNN
-F 1 "GND" H 2005 4827 50  0000 C CNN
-F 2 "" H 2000 5000 50  0001 C CNN
-F 3 "" H 2000 5000 50  0001 C CNN
-	1    2000 5000
+P 1400 5100
+F 0 "#PWR0150" H 1400 4850 50  0001 C CNN
+F 1 "GND" H 1405 4927 50  0000 C CNN
+F 2 "" H 1400 5100 50  0001 C CNN
+F 3 "" H 1400 5100 50  0001 C CNN
+	1    1400 5100
 	1    0    0    -1
 $EndComp
@@
 Wire Wire Line
 	3800 5300 4200 5300
-Text Notes 1300 4800 0    37   ~ 0
+Text Notes 1000 4700 0    37   ~ 0
 I_chg=1.2V / R_chg*100000=0.6A
 Wire Wire Line
@@
 	1    0    0    -1
 $EndComp
+$Comp
+L Switch:SW_MEC_5E SW3
+U 1 1 61F77ED3
+P 1900 5300
+F 0 "SW3" H 1900 5685 50  0000 C CNN
+F 1 "SW_MEC_5E" H 1900 5594 50  0000 C CNN
+F 2 "PSLab:button_SPST_3x4x2.5" H 1900 5600 50  0001 C CNN
+F 3 "http://www.apem.com/int/index.php?controller=attachment&id_attachment=1371" H 1900 5600 50  0001 C CNN
+	1    1900 5300
+	1    0    0    -1
+$EndComp
+Wire Wire Line
+	2300 5100 2100 5100
+Wire Wire Line
+	2100 5100 2100 5200
+Connection ~ 2100 5200
+Wire Wire Line
+	2100 5200 2100 5300
+Wire Wire Line
+	1700 5200 1700 5300
+$Comp
+L power:GND #PWR0103
+U 1 1 62053B95
+P 1700 5300
+F 0 "#PWR0103" H 1700 5050 50  0001 C CNN
+F 1 "GND" H 1705 5127 50  0000 C CNN
+F 2 "" H 1700 5300 50  0001 C CNN
+F 3 "" H 1700 5300 50  0001 C CNN
+	1    1700 5300
+	1    0    0    -1
+$EndComp
+Connection ~ 1700 5300
+Wire Wire Line
+	1400 4700 2200 4700
+Wire Wire Line
+	2200 4700 2200 4800
+Wire Wire Line
+	2200 4800 2300 4800
+Wire Wire Line
+	2300 5000 2200 5000
+Wire Wire Line
+	2200 5000 2200 4900
+Wire Wire Line
+	2200 4900 2100 4900
+Wire Wire Line
+	2100 4900 2100 4800
+Wire Wire Line
+	2100 4800 1700 4800
+Wire Wire Line
+	1700 4800 1700 4900
+$Comp
+L Device:R_Small R63
+U 1 1 62134A7C
+P 1500 5000
+F 0 "R63" H 1559 5046 50  0000 L CNN
+F 1 "51k" H 1559 4955 50  0000 L CNN
+F 2 "Resistor_SMD:R_0603_1608Metric" H 1500 5000 50  0001 C CNN
+F 3 "~" H 1500 5000 50  0001 C CNN
+	1    1500 5000
+	1    0    0    -1
+$EndComp
+Wire Wire Line
+	1500 4900 1700 4900
+Wire Wire Line
+	1400 4900 1400 5100
+Wire Wire Line
+	1400 5100 1500 5100
+Connection ~ 1400 5100
 $EndSCHEMATC

Commit message: Add battery socket, add SW3
Parts:
- added BT3: Battery_Cell, PSLab:2.0mm_connector_edge, symbol Device:Battery_Cell
- R22, R23: Description 1/16W 5% -> 1/16W 1%
- renumbered SW3 to P2
Connections:
- wire segments 509 -> 460
Other:
- moved on the sheet: C22, C23, C24, C25, C26, C27, C28, C29, C31, C32, C39, C41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

Commit message: refactor: replace PGA MAX6S@! with TL082 and MAX5400
Parts:
- removed R22, R23, R28, R29: 10K, Resistor_SMD:R_0603_1608Metric, symbol Device:R
- removed U13, U14: MCP6S21, Package_SO:SOIC-8_3.9x4.9mm_P1.27mm, symbol PSLab:MCP6S21
- added R22, R23, R28, R29: 10k, Resistor_SMD:R_0603_1608Metric, symbol Device:R_Small
- added U13, U14: MAX5400, Package_TO_SOT_SMD:SOT-23-8, symbol PSLab:MAX5400
- added unit 1 of U18
- added unit 3 of U18
- added unit 2 of U8
- renumbered U8 to U18
Connections:
- wire segments 460 -> 464
Other:
- moved on the sheet: C23, C25, C28, C29, C31, C41, R16, R17, R20, R24, R30, R34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

Commit message: refactor: replace MCP4728 with 2 MPC4822
Parts:
- removed U12: MCP4728, Package_SO:MSOP-10_3x3mm_P0.5mm, symbol Analog_DAC:MCP4728
- added R64, R65, R66, R70, R71: 10k, Resistor_SMD:R_0603_1608Metric, symbol Device:R_Small
- added U12: 4051, symbol 4xxx:4051
- added U19, U20: MCP4822, symbol Analog_DAC:MCP4822
Connections:
- net labels added: CS1, CS2, CS3, CS4
- wire segments 464 -> 460
- no-connect marks 31 -> 30
Other:
- moved on the sheet: BT3, C11, C14, C24, C27, C32, C34, C37, C42, C45, J11, J8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

Commit message: Temp6
Parts:
- removed U12: 4051, symbol 4xxx:4051
- added U12: 74HC4051, Package_SO:TSSOP-16_4.4x5mm_P0.65mm, symbol 74xx:74HC4051
- U18, U19, U20: footprint (none) -> Package_SO:SOIC-8_3.9x4.9mm_P1.27mm
Connections:
- net CS.CH1: now also U12.11 (S0)
- net CS.CH2: now also U12.10 (S1)
- net CS.CH3: now also U12.9 (S2); no longer P1.2 (CS)
- net CS1: now also U12.13 (A0)
- net CS2: now also U12.14 (A1)
- net CS3: now also U12.15 (A2)
- net CS4: now also U12.12 (A3)
- net GND: now also U9.5 (+), U12.3 (A), U12.6 (~E), U12.7 (VEE), U12.8 (GND); no longer U9.3 (+)
- net SPI.CS: now also U12.1 (A4); no longer U3.37 (SDA1|RPI52|RC4)
- net VDDA: now also U12.16 (VCC)
- net at U14.7 (W): now also U9.2 (-); no longer U9.6 (-)
- net at R28.1, U14.8 (H): now also U9.1; no longer U9.7
- net at C29.1, R30.1: now also U9.3 (+), U9.7; no longer U9.1, U9.5 (+)
- net at C29.2, R30.2, R34.1: now also U9.6 (-); no longer U9.2 (-)
- new net SD.CS: P1.2 (CS), U12.5 (A5)
Other:
- moved on the sheet: C28, C31, C41, R64, R65, R66, R71, U18A, U18C, U9A, U9B, U9C
