File: schematics/PSLab.kicad_pcb (KiCad board)
At the start: 4 copper layers, 99 x 53.3 mm, 186 parts, among them J1 DoublePins, J11 Li-Ion Battery, J2 Power Pins, J3 Wave Generator, J4 I2C, J5 I2C, J6 ESP01, J7 UART, J8 Battery Switch, J9 SPI, P1 SDCard, Q1 MMBT3906, Q2 MMBT3904, Q3 MMBT3906, Q4 Q_NMOS_DGS, SW1 BOOT, SW2 MCLR Reset, SW3 USB_C - Generic, U1 LDFM33PUR, U10 TL082, U11 TL082, U12 MCP4728, U13 MCP6S21, U14 MCP6S21, U15 CP2102N, U16 SP0503BAHT, U18 LTC4040, U19 TC1240A, U2 74HC126, U3 PIC24EP256GP204, U4 DS1307Z+, U5 TC7660, U7 LM324, U8 TL082, U9 TL082, X2 32.768 kHz, Y1 12 MHz

Commit message: Temp
Parts:
- removed C46: 10uF, Capacitor_SMD:C_0603_1608Metric
- removed C47: 100uF, Capacitor_Tantalum_SMD:CP_EIA-6032-28_Kemet-C
- removed Q4: Q_NMOS_DGS, PSLab:PowerPAK_SO-8_Single
- removed R63: 1690K, Resistor_SMD:R_0603_1608Metric
- removed R64: 324K, Resistor_SMD:R_0603_1608Metric
- removed R65: 178K, Resistor_SMD:R_0603_1608Metric
- removed R66: 60K4, Resistor_SMD:R_0603_1608Metric
- removed U18: LTC4040, PSLab:LTC4040
- removed U19: TC1240A, Package_TO_SOT_SMD:SOT-23-6
- added D7: K1N5817HW-7-F, Diode_SMD:D_SOD-123, F.Cu at (120.3, 83.6)
- added L3: 3.3uH, Inductor_SMD:L_0603_1608Metric, F.Cu at (116.7, 85.0)
- added R68: 470k, Resistor_SMD:R_0603_1608Metric, F.Cu at (117.3, 78.2)
- added R69: 30k, Resistor_SMD:R_0603_1608Metric, F.Cu at (114.1, 78.2)
- added U17: IP5189T, Package_DFN_QFN:QFN-24-1EP_4x4mm_P0.5mm_EP2.6x2.6mm, F.Cu at (121.3, 105.6)
- added U6: HT7333-A, Package_TO_SOT_SMD:SOT-89-3, F.Cu at (97.7, 56.0)
- C11, C14: value 100uF -> 22uF; footprint Capacitor_Tantalum_SMD:CP_EIA-6032-28_Kemet-C -> Capacitor_SMD:C_0603_1608Metric
- C12: value 33uF -> 100uF
- C45: value 2.2uF -> 22uF
- L2: value 2.2uH -> 4.7uH; footprint Inductor_SMD:L_Coilcraft_XAL5030 -> Inductor_SMD:L_0603_1608Metric
- R4: value 18 -> 100k
- R61: value 2K -> 200k
- R62: value 6m -> 0.5R
- U1: value LDFM33PUR -> FP6291; footprint PSLab:DFN-6-1EP_3x3mm_P0.95mm_EP1.7x2.6mm -> Package_TO_SOT_SMD:SOT-23-6
- U5: value TC7660 -> TP7660H
- Z9: value Val** -> Silk
- moved C14 27.9 mm to (122.7, 110.6)
- moved C11 27.2 mm to (116.7, 104.6), turned to 90 degrees
- moved U1 26.4 mm to (116.6, 81.4)
- moved L2 13.8 mm to (124.8, 105.2)
- moved R61 12.8 mm to (125.3, 108.6), turned to 90 degrees
- moved R4 10.8 mm to (113.7, 83.2)
- moved C45 10.6 mm to (117.3, 110.6), turned to 90 degrees
- moved C12 6.26 mm to (120.7, 78.4), turned to 90 degrees
- moved R62 1.19 mm to (119.9, 110.0)
Connections:
- net /_BATT renamed Net-(J11-Pad2)
- C11 pad 1: /DBL -> Net-(C11-Pad1)
- C14 pad 2: Net-(C14-Pad2) -> GND
- C45 pad 1: /VINPUT -> /BAT+
- J8 pad 2: /BATT -> /BAT+
- L2 pad 1: /BATT -> Net-(L2-Pad1)
- L2 pad 2: /L2 -> Net-(C14-Pad1)
- R4 pad 1: /DBL -> Net-(R4-Pad1)
- R4 pad 2: +10V -> GND
- R62 pad 1: /VINPUT -> /BAT+
- R62 pad 2: /CLN -> Net-(C14-Pad1)
- U1 pad 1: +3V3 -> Net-(D7-Pad2)
- U1 pad 2: (no net) -> GND
- U1 pad 3: (no net) -> Net-(R68-Pad2)
- U1 pad 4: GND -> +5V
- U1 pad 6: +5V -> Net-(R4-Pad1)
- U5 pad 8: /DBL -> +10V
Routing:
- net +5V: track 183.4 -> 123.6 mm, vias 8 -> 4
- net /VINPUT: track 77.1 -> 48.4 mm, vias 4 -> 2
- net /BATT: track 26.1 -> 0.00 mm
- net Net-(R63-Pad2): track 24.3 -> 0.00 mm, vias 2 -> 0
- net /BAT+: track 0.00 -> 18.6 mm
- net /CLN: track 15.7 -> 0.00 mm, vias 2 -> 0
- net /DBL: track 13.7 -> 0.00 mm
- net +10V: track 81.1 -> 93.9 mm
- net Net-(C14-Pad2): track 7.45 -> 0.00 mm
- net /PFI: track 7.22 -> 0.00 mm
- net Net-(D7-Pad2): track 0.00 -> 6.07 mm
- net Net-(R61-Pad1): track 5.10 -> 0.00 mm
- net Net-(R68-Pad2): track 0.00 -> 4.30 mm
- net Net-(C14-Pad1): track 3.69 -> 0.00 mm
- net GND: track 206.4 -> 202.8 mm, vias 70 -> 65
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- removed copper zone on F.Cu, net /BATT
- removed copper zone on F.Cu, net /L2
Other:
- net class Default: clearance 0.156 -> 0.15; trace_width 0.3048 -> 0.15; via_dia 0.9144 -> 0.7; via_drill 0.4064 -> 0.4
- rule trace_clearance: 0.156 -> 0.15
- rule trace_min: 0.2 -> 0.15
- rule via_min_drill: 0.3048 -> 0.4
- rule via_min_size: 0.4 -> 0.6

Commit message: Temp2
Parts:
- L2: footprint Inductor_SMD:L_0603_1608Metric -> Inductor_SMD:L_Taiyo-Yuden_MD-2020
- moved U6 48.9 mm to (113.3, 102.4), turned to 270 degrees
- moved C20 44.7 mm to (116.9, 101.4)
- moved C15 39.1 mm to (109.7, 101.2)
- moved Z10 15.1 mm to (113.7, 89.2)
- moved F1 14.5 mm to (100.5, 82.6), turned to 0 degrees
- moved R61 7.78 mm to (122.9, 101.2), turned to 180 degrees
- moved L2 4.57 mm to (123.5, 109.6), turned to 180 degrees
- moved C14 2.24 mm to (120.7, 111.6), turned to 180 degrees
- moved C11 0.57 mm to (117.1, 105.0)
- moved R5 0.36 mm to (123.2, 82.0)
- moved C12 0.20 mm to (120.5, 78.4)
Routing:
- net +5V: track 123.6 -> 153.8 mm, vias 4 -> 8
- net /BAT+: track 18.6 -> 34.1 mm
- net GND: track 202.8 -> 215.2 mm, vias 65 -> 70
- net Net-(R61-Pad1): track 0.00 -> 12.1 mm, vias 0 -> 2
- net +3V3: track 251.4 -> 262.8 mm
- net Net-(L2-Pad1): track 0.00 -> 7.79 mm
- net Net-(C14-Pad1): track 0.00 -> 5.19 mm
- net RxD2: track 62.4 -> 60.9 mm
- net /VUSBIN: track 14.2 -> 15.3 mm
- net TxD2: track 44.1 -> 43.1 mm
- net /VINPUT: track 48.4 -> 48.7 mm, vias 2 -> 4
Other:
- net class Default: via_dia 0.7 -> 0.5; via_drill 0.4 -> 0.3
- rule via_min_drill: 0.4 -> 0.3
- rule via_min_size: 0.6 -> 0.5

Commit message: Temp3
Parts:
- SW3: footprint Connector_USB:USB_C_Receptacle_XKB_U262-16XN-4BVC11 -> incremental_library:USB_C_Receptacle_12pin_SMT
- moved C2 26.6 mm to (105.8, 105.7), turned to 180 degrees
- moved U16 20.1 mm to (80.7, 75.2)
- moved R60 19.2 mm to (99.5, 64.0), turned to 180 degrees
- moved R59 16.9 mm to (100.2, 66.0), turned to 180 degrees
- moved F1 2.12 mm to (102.5, 81.9), turned to 270 degrees
- moved D4 0.92 mm to (93.8, 66.4)
- moved Z2 0.80 mm to (99.4, 78.8)
- moved Z3 0.80 mm to (99.4, 72.1)
- moved Z4 0.80 mm to (99.4, 76.6)
- moved Z5 0.80 mm to (99.4, 74.4)
- moved R53 0.67 mm to (95.9, 66.7)
- turned R58 to 270 degrees
Routing:
- net /D-: track 20.4 -> 7.50 mm
- net /D+: track 19.5 -> 8.24 mm
- net /CC1: track 10.8 -> 0.00 mm
- net /VBusSense: track 10.9 -> 2.16 mm
- net /CC2: track 8.44 -> 0.00 mm
- net /VUSBIN: track 15.3 -> 10.8 mm
- net /UARTReset: track 3.02 -> 0.01 mm
- net GND: track 215.2 -> 213.2 mm
- net /VINPUT: track 48.7 -> 49.4 mm
- net +3V3: track 262.8 -> 262.0 mm, vias 5 -> 4
- added copper zone on F.Cu, net GND
- removed copper zone on F.Cu, net /VUSBIN

Commit message: Temp4
Parts:
- L1: footprint Inductor_SMD:L_0603_1608Metric -> Inductor_SMD:L_Taiyo-Yuden_MD-2020
- L3: value 3.3uH -> 4.7uH; footprint Inductor_SMD:L_0603_1608Metric -> Inductor_SMD:L_Taiyo-Yuden_MD-2020
- U15: value CP2102N -> CP2102N-xxx-xQFN20x; footprint Package_DFN_QFN:QFN-24-1EP_4x4mm_P0.5mm_EP2.6x2.6mm -> PSLab:QFN-20_EP_3x3_Pitch0.5mm
- moved U16 23.5 mm to (104.2, 75.5)
- moved U15 3.04 mm to (109.2, 74.9)
- moved C43 2.01 mm to (110.1, 68.3), turned to 180 degrees
- moved SW3 1.20 mm to (94.0, 75.5)
- moved Z2 1.20 mm to (100.6, 78.8)
- moved Z3 1.20 mm to (100.6, 72.1)
- moved Z4 1.20 mm to (100.6, 76.6)
- moved Z5 1.20 mm to (100.6, 74.4)
- moved C44 0.70 mm to (110.1, 70.0), turned to 180 degrees
- moved L3 0.28 mm to (116.9, 84.8)
- moved F1 0.20 mm to (102.5, 81.7)
Connections:
- net /UARTReset renamed Net-(R51-Pad1)
- C43 pad 1: +3V3 -> /CP2102_Vreg
- C44 pad 1: +3V3 -> /CP2102_Vreg
- R51 pad 2: +3V3 -> /CP2102_Vreg
- R54 pad 1: /MRxD -> Net-(R54-Pad1)
- R55 pad 1: /MTxD -> Net-(R55-Pad1)
- U15 pad 12: (no net) -> GND
- U15 pad 17: (no net) -> Net-(R54-Pad1)
- U15 pad 18: (no net) -> Net-(R55-Pad1)
- U15 pad 2: GND -> (no net)
- U15 pad 20: /MRxD -> (no net)
- U15 pad 21: /MTxD -> GND
- U15 pad 3: /D+ -> GND
- U15 pad 4: /D- -> /D+
- U15 pad 5: +3V3 -> /D-
- U15 pad 6: +3V3 -> /CP2102_Vreg
- U15 pad 7: +3V3 -> +5V
Routing:
- net +3V3: track 262.0 -> 241.9 mm
- net /D-: track 7.50 -> 26.9 mm
- net GND: track 213.2 -> 230.5 mm, vias 70 -> 112
- net /D+: track 8.24 -> 25.4 mm
- net /CC2: track 0.00 -> 13.8 mm, vias 0 -> 2
- net /CC1: track 0.00 -> 12.6 mm, vias 0 -> 2
- net /CP2102_Vreg: track 0.00 -> 12.3 mm
- net Net-(R54-Pad1): track 0.00 -> 11.0 mm
- net +5V: track 154.3 -> 164.6 mm, vias 8 -> 9
- net /VUSBIN: track 10.8 -> 21.1 mm
- net /MRxD: track 9.06 -> 0.00 mm
- net /VBusSense: track 2.16 -> 9.56 mm, vias 0 -> 2
- net Net-(R55-Pad1): track 0.00 -> 6.81 mm
- net /MTxD: track 4.55 -> 0.00 mm
- net Net-(R51-Pad1): track 0.01 -> 4.49 mm
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
Commit message: Temp5
Parts:
- removed D6: LL4148, Diode_SMD:D_MiniMELF
- removed TP3: TEST, PSLab:Voltage_Test_Point
Connections:
- D5 pad 1: Net-(D5-Pad1) -> +5V
Routing:
- net -10V: track 123.5 -> 110.5 mm, vias 6 -> 8
- net GND: track 230.5 -> 241.2 mm, vias 112 -> 144
- net Net-(D5-Pad1): track 8.87 -> 0.00 mm
- net +5V: track 164.6 -> 171.3 mm
- net Net-(R54-Pad1): track 11.0 -> 5.71 mm, vias 0 -> 2
- net +6V: track 112.8 -> 109.9 mm
- net -6V: track 91.7 -> 89.7 mm
- net +3V3: track 241.9 -> 243.9 mm
- net SCK: track 121.1 -> 119.5 mm
- net VDDA: track 113.9 -> 115.5 mm
- net SDO: track 116.6 -> 115.5 mm
- net Net-(U14-Pad3): track 19.1 -> 20.0 mm
- removed copper zone on B.Cu, net (none)
- removed copper zone on F.Cu, net (none)
- removed copper zone on L3.Power, net (none)
