File: schematics/PSLab.kicad_sch (KiCad schematic)
At the start: 212 parts, among them J1 DoublePins, J10 Programmer, J2 Power Pins, J3 Wave Generator, J4 I2C, J5 I2C, J6 ESP01, J7 UART, J8 Micro_SD_Card_Det_9_pin, J9 SPI, P2 USB_C - Generic, Q1 MMBT3906, Q2 MMBT3904, Q3 MMBT3906, SW1 SW_MEC_5E, SW2 SW_MEC_5E, SW3 SW_MEC_5E, U1 FP6291, U10 TL082, U11 TL082, U12 74HC4051, U13 MAX5400, U14 MAX5400, U15 CP2102N-xxx-xQFN20x, U16 SP0503BAHT, U17 MT1470, U18 TL082, U19 MCP4822, U2 74HC126, U20 MCP4822, U21 IP5189T, U3 PIC24EP256GP204, U4 DS1307Z+T&R, U5 TP7660H, U6 HT7333-A, U7 LM324, U8 LM833, U9 TL082, X2 32.768 kHz, Y1 12MHz

Commit message: chore: modify descriptions and silk screens
Parts:
- C23, C29: value 1pF -> 0.5pF
- R11, R27, R36, R47, R5, R51: value 1K -> 1k
- R40, R46, R50: value 200K -> 200k
- renumbered BT3 to J11, P2 to J12, BT1 to J13, Y1 to X1, BT2 to Z1
Other:
- moved on the sheet: C34, C37, U11C

Commit message: 20220608
Parts:
- removed C28, C31, C41: 100nF, Capacitor_SMD:C_0603_1608Metric, symbol Device:C
- removed C29: 0.5pF, Capacitor_SMD:C_0603_1608Metric, symbol Device:C
- removed J2: Power Pins, Connector_PinSocket_2.54mm:PinSocket_1x08_P2.54mm_Vertical, symbol Connector_Generic:Conn_01x08
- removed J3: Wave Generator, Connector_PinSocket_2.54mm:PinSocket_1x08_P2.54mm_Vertical, symbol Connector_Generic:Conn_01x08
- removed J4, J5: I2C, Connector_PinSocket_2.54mm:PinSocket_1x04_P2.54mm_Vertical, symbol Connector_Generic:Conn_01x04
- removed J7: UART, Connector_PinSocket_2.54mm:PinSocket_1x04_P2.54mm_Vertical, symbol Connector_Generic:Conn_01x04
- removed J9: SPI, Connector_PinSocket_2.54mm:PinSocket_1x06_P2.54mm_Vertical, symbol Connector_Generic:Conn_01x06
- removed R23, R28: 10k, Resistor_SMD:R_0603_1608Metric, symbol Device:R_Small
- removed R4: 100k, Resistor_SMD:R_0603_1608Metric, symbol Device:R_Small
- removed U1: FP6291, Package_TO_SOT_SMD:SOT-23-6, symbol PSLab:FP6291
- removed U18: TL082, Package_SO:SOIC-8_3.9x4.9mm_P1.27mm, symbol Amplifier_Operational:TL082
- removed U6: HT7333-A, Package_TO_SOT_SMD:SOT-89-3, symbol Regulator_Linear:HT75xx-1-SOT89
- added C5: 10nF, Capacitor_SMD:C_0603_1608Metric, symbol Device:C
- added J2: Conn_01x25, Connector_PinHeader_2.54mm:PinHeader_1x25_P2.54mm_Vertical, symbol Connector_Generic:Conn_01x25
- added J3: Conn_01x13, Connector_PinHeader_2.54mm:PinHeader_1x13_P2.54mm_Vertical, symbol Connector_Generic:Conn_01x13
- added R78, R79: 3k, Resistor_SMD:R_0603_1608Metric, symbol Device:R
- added R? (x2): R_Small, symbol Device:R_Small
- added R?: 100, symbol Device:R_Small
- added R?: 125k, symbol Device:R_Small
- added R?: 40k, symbol Device:R_Small
- added R?: 120k, symbol Device:R_Small
- added R?: 500k, symbol Device:R_Small
- added R?: 60k, symbol Device:R_Small
- added U1: AP3015A, Package_TO_SOT_SMD:SOT-23-5, symbol PSLab:AP3015A
- added U6: AMS1117-3.3, Package_TO_SOT_SMD:SOT-223-3_TabPin2, symbol Regulator_Linear:AMS1117-3.3
- added U?: CD4051B, symbol Analog_Switch:CD4051B
- C23: value 0.5pF -> 10nF; Mfr No. VJ0603A0R5BXJCW1BC -> C0603C104J4RACTU; PartNumber VJ0603A0R5BXJCW1BC -> C0603C104J4RACTU; Price 0.45 -> 0.15
- D8, D9: footprint Diode_SMD:D_SOD-123 -> Diode_SMD:D_MiniMELF
Connections:
- net +3V3: now also J2.13 (Pin_13), J2.6 (Pin_6), J2.9 (Pin_9), U6.2 (VO)
- net +5V: now also J3.1 (Pin_1), U1.4 (EN), U1.5 (VIN), U6.3 (VI)
- net +6V: now also U?.16 (VDD)
- net -6V: now also U?.7 (VEE)
- net CH1_IN: now also U13.7 (W), U8.7
- net CH2: now also R34.1; no longer R34.2
- net CH2_IN: now also U14.7 (W), U8.1
- net GND: now also C23.2, C5.2, J2.14 (Pin_14), J2.18 (Pin_18), J2.20 (Pin_20), J2.22 (Pin_22), J2.24 (Pin_24), J2.5 (Pin_5), J2.8 (Pin_8), J3.13 (Pin_13), J3.2 (Pin_2), J3.8 (Pin_8), U1.2 (GND), U6.1 (GND), U?.8 (VSS)
- net OSC_REF1: now also R16.1, R17.1, C5.1
- net OSC_REF2: now also C23.1, R22.1, R29.1
- net PCS: now also J2.25 (Pin_25)
- net PVS1: now also J2.23 (Pin_23)
- net PVS2: now also J2.21 (Pin_21)
- net PVS3: now also J2.19 (Pin_19)
- net RxD2: now also J3.4 (Pin_4)
- net SCK: now also J2.3 (Pin_3)
- net SCL: now also J2.11 (Pin_11), J2.15 (Pin_15)
- net SDA: now also J2.10 (Pin_10), J2.16 (Pin_16)
- net SDI: now also J2.2 (Pin_2)
- net SDO: now also J2.4 (Pin_4)
- net SINE1: now also J3.6 (Pin_6)
- net SINE2: now also J3.7 (Pin_7)
- net SPI.CS: now also J2.1 (Pin_1)
- net SQR1: now also J3.9 (Pin_9)
- net SQR2: now also J3.10 (Pin_10)
- net SQR3: now also J3.11 (Pin_11)
- net SQR4: now also J3.12 (Pin_12)
- net TxD2: now also J3.3 (Pin_3)
- net at U8.6 (-): now also U13.8 (H), R78.2; no longer U14.7 (W)
- net at U14.8 (H): now also U8.2 (-), R79.2; no longer U8.7
- net at D7.2 (A), L3.2: now also U1.1 (SW)
- net at R68.2, R69.1: now also U1.3 (FB)
- net at R20.1, R24.1: now also U9.6 (-); no longer C23.2, U9.2 (-)
- new net: R30.1, R79.1, U9.1
- new net: R30.2, R34.2, U9.2 (-)
- new net: R20.2, R78.1, U9.7
- new net: R?.1, R?.2 (x7)
- now unconnected: U13.1 (L), U14.1 (L)
- no-connect marks 27 -> 26
Other:
- moved on the sheet: C2, C25, J1, J10, J6, R16, R17, R20, R22, R24, R29, R30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

Commit message: chore: remove 7660
Parts:
- removed C16, C19: 33uF, Capacitor_Tantalum_SMD:CP_EIA-3528-21_Kemet-B, symbol Device:CP1
- removed C22, C26: 100nF, Capacitor_SMD:C_0603_1608Metric, symbol Device:C
- removed CB2: CircuitBreaker_1P, Jumper:SolderJumper-2_P1.3mm_Open_RoundedPad1.0x1.5mm, symbol Device:CircuitBreaker_1P
- removed R? (x2): R_Small, symbol Device:R_Small
- removed R?: 100, symbol Device:R_Small
- removed R?: 125k, symbol Device:R_Small
- removed R?: 40k, symbol Device:R_Small
- removed R?: 120k, symbol Device:R_Small
- removed R?: 500k, symbol Device:R_Small
- removed R?: 60k, symbol Device:R_Small
- removed U13, U14: MAX5400, Package_TO_SOT_SMD:SOT-23-8, symbol PSLab:MAX5400
- removed U5: TP7660H, Package_SO:SOIC-8_3.9x4.9mm_P1.27mm, symbol PSLab:TP7660H
- removed U8: LM833, Package_SO:SOIC-8_3.9x4.9mm_P1.27mm, symbol Amplifier_Operational:TL082
- removed U?: CD4051B, symbol Analog_Switch:CD4051B
- added R23, R4: 10k, Resistor_SMD:R_0603_1608Metric, symbol Device:R_Small
- added U13: TL082, Package_SO:SOIC-8_3.9x4.9mm_P1.27mm, symbol Amplifier_Operational:TL082
- added U14, U18: MCP6S21-I/SN, Package_SO:SOIC-8_3.9x4.9mm_P1.27mm, symbol PSLab:MCP6S21
- J13: footprint PSLab:BatteryHolder_LINX_BAT-HLD-012-SMT -> PSLab:BatteryHolder_A359
- R20, R30: value 100k -> 200k
- R68: value 130k -> 180k
- R69: value 10k -> 30k
- R78, R79: value 3k -> 10k
Connections:
- net +6V: now also U13.8 (V+)
- net -6V: now also U13.4 (V-)
- net CH1_IN: now also U14.1 (OUT)
- net CH2_IN: now also U18.1 (OUT)
- net CS1: now also U14.5 (CS)
- net CS2: now also U18.5 (CS)
- net GND: now also U9.3 (+), U9.5 (+), U14.4 (GND), U18.4 (GND)
- net OSC_REF1: now also U13.6 (-), U13.7, U14.3 (VREF), U18.3 (VREF); no longer C5.1, R16.1, R17.1
- net OSC_REF2: no longer U9.3 (+), U9.5 (+)
- net SCK: now also U14.7 (SCK), U18.7 (SCK)
- net SDO: now also U14.6 (SDI), U18.6 (SDI)
- net VDDA: now also R23.1, R4.1, U14.8 (VDD), U18.8 (VDD)
- net at R79.2: now also R23.2, U18.2 (CHA)
- net at R78.2: now also R4.2, U14.2 (CHA)
- net at R30.1, R79.1: now also U9.7; no longer U9.1
- net at R30.2, R34.2: now also U9.6 (-); no longer U9.2 (-)
- net at R20.1, R24.1: now also U9.2 (-); no longer U9.6 (-)
- net at R20.2, R78.1: now also U9.1; no longer U9.7
- net +10V renamed +9V
- net -10V renamed -9V
- new net: C5.1, R16.1, R17.1, U13.3 (+), U13.5 (+)
- new net: U13.1, U13.2 (-)
- no-connect marks 26 -> 25
Other:
- note added: "I_chg=100000 * 1.2V / R_chg =0.6A"
- note added: "Voltage Doubler"
- note added: "Voltage Inverter Regulator"
- note added: "Vout=1.23*210k/30k=8.61V"
- note removed: "I_chg=1.2V / R_chg*100000=0.6A"
- note removed: "Over Current set to 48000/100k=0.48A"
- note removed: "Voltage Doubler and Inverter"
- note removed: "Voltage Regulator"
- note removed: "Vout=0.6*140k/10k=8.4V"
- moved on the sheet: C39, U9A, U9B, U9C

Commit message: refactor: send to manufacturer
Parts:
- removed CB1: CircuitBreaker_1P, Jumper:SolderJumper-2_P1.3mm_Bridged_RoundedPad1.0x1.5mm, symbol Device:CircuitBreaker_1P
- removed D6: GREEN, LED_SMD:LED_0805_2012Metric, symbol Device:LED_ALT
- removed R13, R65: 10k, Resistor_SMD:R_0603_1608Metric, symbol Device:R_Small
- removed R27: 1k, Resistor_SMD:R_0603_1608Metric, symbol Device:R
- removed R62: 0.5R, Resistor_SMD:R_0603_1608Metric, symbol Device:R_Small
- removed R74: 1k, Resistor_SMD:R_0603_1608Metric, symbol Device:R_Small
- removed U19: MCP4822, Package_SO:SOIC-8_3.9x4.9mm_P1.27mm, symbol Analog_DAC:MCP4822
- added D10, D11, D12, D13: White, LED_SMD:LED_0603_1608Metric, symbol Device:LED_Small
Connections:
- net DAC.1 is gone; now on net PVS3: U20.8 (VA), U7.3 (+)
- net DAC.4 is gone; now on net DAC.2: U7.10 (+)
- net -9V: now also C51.2, C54.2, R76.2, U17.1 (GND)
- net BAT+: now also C14.1, U21.9 (VBAT)
- net LD3: now also D10.1 (K), D11.2 (A), D12.1 (K), D13.2 (A); no longer U21.24 (L1)
- net LD2: now reaches U21.1 (L2)
- net LD2: now also D10.2 (A), D11.1 (K)
- net CS4: no longer names the net of U12.12 (A3)
- new net LD1: D12.2 (A), D13.1 (K), U21.24 (L1)
Other:
- moved on the sheet: C24, C27, C32, R18, R19, R25, R26, R35, R37, U7A, U7B, U7D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
